Commit message: Urdf is so irritating

File: src/micromouse_description/urdf/micromouse.urdf (robot description, URDF)
Before this commit: robot micromouse, 10 links, 9 joints
Links:
- removed link wheel_left_back
- removed link wheel_left_front
- removed link wheel_right_back
- removed link wheel_right_front
- added link wheel_left, mass 0.05; collision cylinder length=0.02 radius=0.03; visual cylinder length=0.02 radius=0.03
- added link wheel_right, mass 0.05; collision cylinder length=0.02 radius=0.03; visual cylinder length=0.02 radius=0.03
- link ir_front: geometry collision cylinder length=0.02 radius=0.005; visual cylinder length=0.02 radius=0.005
- link ir_front_left: geometry collision cylinder length=0.02 radius=0.005; visual cylinder length=0.02 radius=0.005
- link ir_front_right: geometry collision cylinder length=0.02 radius=0.005; visual cylinder length=0.02 radius=0.005
- link ir_left: geometry collision cylinder length=0.02 radius=0.005; visual cylinder length=0.02 radius=0.005
- link ir_right: geometry collision cylinder length=0.02 radius=0.005; visual cylinder length=0.02 radius=0.005
Joints:
- removed joint wheel_left_back_joint
- removed joint wheel_left_front_joint
- removed joint wheel_right_back_joint
- removed joint wheel_right_front_joint
- added joint wheel_left_joint: type continuous, parent base_link, child wheel_left, origin xyz=0 0.04 -0.02 rpy=0 0 0, axis 0 1 0
- added joint wheel_right_joint: type continuous, parent base_link, child wheel_right, origin xyz=0 -0.04 -0.02 rpy=0 0 0, axis 0 1 0

File: src/micromouse_description/urdf/micromouse.urdf.xacro (robot description, xacro)
@@ -7,4 +7,5 @@
   <xacro:property name="robot_length" value="0.12"/>
   <xacro:property name="robot_width" value="0.10"/>
+  <xacro:property name="robot_height" value="0.04"/>
   <xacro:property name="sensor_range" value="0.10"/>
   <!-- ========= Base Link ========= -->
@@ -12,5 +13,5 @@
     <visual>
       <geometry>
-        <box size="${robot_length} ${robot_width} 0.04"/>
+        <box size="${robot_length} ${robot_width} ${robot_height}"/>
       </geometry>
       <material name="Blue"/>
@@ -18,5 +19,5 @@
     <collision>
       <geometry>
-        <box size="${robot_length} ${robot_width} 0.04"/>
+        <box size="${robot_length} ${robot_width} ${robot_height}"/>
       </geometry>
     </collision>
@@ -27,5 +28,4 @@
   </link>
   <!-- ========= Wheels ========= -->
-  <!-- Left Wheels -->
   <xacro:macro name="wheel" params="name x y z">
     <link name="${name}">
@@ -53,11 +53,8 @@
     </joint>
   </xacro:macro>
-  <!-- Left wheels -->
-  <xacro:wheel name="wheel_left_front" x="0.03" y="${wheel_separation/2}" z="-0.02"/>
-  <xacro:wheel name="wheel_left_back" x="-0.03" y="${wheel_separation/2}" z="-0.02"/>
-  <!-- Right wheels -->
-  <xacro:wheel name="wheel_right_front" x="0.03" y="-${wheel_separation/2}" z="-0.02"/>
-  <xacro:wheel name="wheel_right_back" x="-0.03" y="-${wheel_separation/2}" z="-0.02"/>
-  <!-- ========= IR Sensors (Ray Sensors) ========= -->
+  <!-- Left and Right wheels -->
+  <xacro:wheel name="wheel_left" x="0" y="${wheel_separation/2}" z="-0.02"/>
+  <xacro:wheel name="wheel_right" x="0" y="-${wheel_separation/2}" z="-0.02"/>
+  <!-- ========= IR Sensors ========= -->
   <xacro:macro name="ir_sensor" params="name x y yaw">
     <link name="${name}">
@@ -68,4 +65,9 @@
         <material name="Red"/>
       </visual>
+      <collision>
+        <geometry>
+          <cylinder radius="0.005" length="0.02"/>
+        </geometry>
+      </collision>
     </link>
     <joint name="${name}_joint" type="fixed">
@@ -77,10 +79,10 @@
   <!-- Front Sensors -->
   <xacro:ir_sensor name="ir_front" x="0.06" y="0" yaw="0"/>
-  <xacro:ir_sensor name="ir_front_left" x="0.05" y="0.03" yaw="0.785"/> <!-- 45 deg -->
-  <xacro:ir_sensor name="ir_front_right" x="0.05" y="-0.03" yaw="-0.785"/> <!-- -45 deg -->
+  <xacro:ir_sensor name="ir_front_left" x="0.05" y="0.03" yaw="0.785"/>
+  <xacro:ir_sensor name="ir_front_right" x="0.05" y="-0.03" yaw="-0.785"/>
   <!-- Side Sensors -->
-  <xacro:ir_sensor name="ir_left" x="0" y="0.05" yaw="1.57"/> <!-- 90 deg -->
-  <xacro:ir_sensor name="ir_right" x="0" y="-0.05" yaw="-1.57"/> <!-- -90 deg -->
-  <!-- ========= Transmission & Diff Drive Plugin ========= -->
+  <xacro:ir_sensor name="ir_left" x="0" y="0.05" yaw="1.57"/>
+  <xacro:ir_sensor name="ir_right" x="0" y="-0.05" yaw="-1.57"/>
+  <!-- ========= Diff Drive Plugin ========= -->
   <gazebo>
     <plugin name="diff_drive_controller" filename="libgazebo_ros_diff_drive.so">
@@ -92,10 +94,14 @@
       <wheelSeparation>${wheel_separation}</wheelSeparation>
       <wheelDiameter>${wheel_radius*2}</wheelDiameter>
-      <leftJoint>wheel_left_front</leftJoint>
-      <rightJoint>wheel_right_front</rightJoint>
-      <leftJoint>wheel_left_back</leftJoint>
-      <rightJoint>wheel_right_back</rightJoint>
+      <leftJoint>wheel_left</leftJoint>
+      <rightJoint>wheel_right</rightJoint>
       <robotBaseFrame>base_link</robotBaseFrame>
     </plugin>
   </gazebo>
+  <inertial>
+  <mass value="0.5"/>
+  <inertia ixx="0.001" ixy="0.0" ixz="0.0"
+           iyy="0.001" iyz="0.0"
+           izz="0.001"/>
+</inertial>
 </robot>

Commit message: Xarco not found error changes

File: src/micromouse_description/urdf/micromouse.urdf (robot description, URDF)
Before this commit: robot micromouse, 8 links, 7 joints
Links:
- link ir_front: mass None -> 0.001
- link ir_front_left: mass None -> 0.001
- link ir_front_right: mass None -> 0.001
- link ir_left: mass None -> 0.001
- link ir_right: mass None -> 0.001

File: src/micromouse_description/urdf/micromouse.urdf.xacro (robot description, xacro)
@@ -7,5 +7,4 @@
   <xacro:property name="robot_length" value="0.12"/>
   <xacro:property name="robot_width" value="0.10"/>
-  <xacro:property name="robot_height" value="0.04"/>
   <xacro:property name="sensor_range" value="0.10"/>
   <!-- ========= Base Link ========= -->
@@ -13,5 +12,5 @@
     <visual>
       <geometry>
-        <box size="${robot_length} ${robot_width} ${robot_height}"/>
+        <box size="${robot_length} ${robot_width} 0.04"/>
       </geometry>
       <material name="Blue"/>
@@ -19,13 +18,15 @@
     <collision>
       <geometry>
-        <box size="${robot_length} ${robot_width} ${robot_height}"/>
+        <box size="${robot_length} ${robot_width} 0.04"/>
       </geometry>
     </collision>
     <inertial>
       <mass value="0.5"/>
-      <inertia ixx="0.001" iyy="0.001" izz="0.001"/>
+      <inertia ixx="0.001" ixy="0.0" ixz="0.0"
+               iyy="0.001" iyz="0.0"
+               izz="0.001"/>
     </inertial>
   </link>
-  <!-- ========= Wheels ========= -->
+  <!-- ========= Wheel Macro ========= -->
   <xacro:macro name="wheel" params="name x y z">
     <link name="${name}">
@@ -43,5 +44,7 @@
       <inertial>
         <mass value="0.05"/>
-        <inertia ixx="0.0001" iyy="0.0001" izz="0.0001"/>
+        <inertia ixx="0.0001" ixy="0.0" ixz="0.0"
+                 iyy="0.0001" iyz="0.0"
+                 izz="0.0001"/>
       </inertial>
     </link>
@@ -53,8 +56,8 @@
     </joint>
   </xacro:macro>
-  <!-- Left and Right wheels -->
+  <!-- ========= Wheels (1 per side) ========= -->
   <xacro:wheel name="wheel_left" x="0" y="${wheel_separation/2}" z="-0.02"/>
   <xacro:wheel name="wheel_right" x="0" y="-${wheel_separation/2}" z="-0.02"/>
-  <!-- ========= IR Sensors ========= -->
+  <!-- ========= IR Sensor Macro ========= -->
   <xacro:macro name="ir_sensor" params="name x y yaw">
     <link name="${name}">
@@ -70,4 +73,10 @@
         </geometry>
       </collision>
+      <inertial>
+        <mass value="0.001"/>
+        <inertia ixx="1e-6" ixy="0" ixz="0"
+                 iyy="1e-6" iyz="0"
+                 izz="1e-6"/>
+      </inertial>
     </link>
     <joint name="${name}_joint" type="fixed">
@@ -79,10 +88,10 @@
   <!-- Front Sensors -->
   <xacro:ir_sensor name="ir_front" x="0.06" y="0" yaw="0"/>
-  <xacro:ir_sensor name="ir_front_left" x="0.05" y="0.03" yaw="0.785"/>
-  <xacro:ir_sensor name="ir_front_right" x="0.05" y="-0.03" yaw="-0.785"/>
+  <xacro:ir_sensor name="ir_front_left" x="0.05" y="0.03" yaw="0.785"/> <!-- 45 deg -->
+  <xacro:ir_sensor name="ir_front_right" x="0.05" y="-0.03" yaw="-0.785"/> <!-- -45 deg -->
   <!-- Side Sensors -->
-  <xacro:ir_sensor name="ir_left" x="0" y="0.05" yaw="1.57"/>
-  <xacro:ir_sensor name="ir_right" x="0" y="-0.05" yaw="-1.57"/>
-  <!-- ========= Diff Drive Plugin ========= -->
+  <xacro:ir_sensor name="ir_left" x="0" y="0.05" yaw="1.57"/> <!-- 90 deg -->
+  <xacro:ir_sensor name="ir_right" x="0" y="-0.05" yaw="-1.57"/> <!-- -90 deg -->
+  <!-- ========= Gazebo Diff Drive Plugin ========= -->
   <gazebo>
     <plugin name="diff_drive_controller" filename="libgazebo_ros_diff_drive.so">
@@ -94,14 +103,8 @@
       <wheelSeparation>${wheel_separation}</wheelSeparation>
       <wheelDiameter>${wheel_radius*2}</wheelDiameter>
-      <leftJoint>wheel_left</leftJoint>
-      <rightJoint>wheel_right</rightJoint>
+      <leftJoint>wheel_left_joint</leftJoint>
+      <rightJoint>wheel_right_joint</rightJoint>
       <robotBaseFrame>base_link</robotBaseFrame>
     </plugin>
   </gazebo>
-  <inertial>
-  <mass value="0.5"/>
-  <inertia ixx="0.001" ixy="0.0" ixz="0.0"
-           iyy="0.001" iyz="0.0"
-           izz="0.001"/>
-</inertial>
 </robot>
